File: Microcontroller_board/Microcontroller.kicad_sch (KiCad schematic)
At the start: 10 parts, among them SW1 Reset, U1 ESP32-WROOM-E

Commit message: Added more pages, CP and RS485
Changed lines of the file:
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@@
     (stroke (width 0) (type default))
   )
-  (text "ESP32" (at 53.34 50.8 0)
+  (text "ESP32" (at 34.29 41.91 0)
     (effects (font (size 7 7) (thickness 1.2) bold italic) (justify left bottom))
   )
-  (label "RX0" (at 189.23 95.25 0) (fields_autoplaced)
-    (effects (font (size 1.27 1.27)) (justify left bottom))
+  (hierarchical_label "EN" (shape input) (at 100.33 48.26 180) (fields_autoplaced)
+    (effects (font (size 1.27 1.27)) (justify right))
   )
-  (label "IO0" (at 189.23 100.33 0) (fields_autoplaced)
-    (effects (font (size 1.27 1.27)) (justify left bottom))
+  (hierarchical_label "TXD_RS485" (shape input) (at 208.28 127 180) (fields_autoplaced)
+    (effects (font (size 1.27 1.27)) (justify right))
   )
-  (label "EN" (at 82.55 92.71 0) (fields_autoplaced)
-    (effects (font (size 1.27 1.27)) (justify left bottom))
+  (hierarchical_label "RX0" (shape input) (at 189.23 95.25 0) (fields_autoplaced)
+    (effects (font (size 1.27 1.27)) (justify left))
   )
-  (label "TX0" (at 189.23 92.71 0) (fields_autoplaced)
-    (effects (font (size 1.27 1.27)) (justify left bottom))
+  (hierarchical_label "LOCK_STATUS" (shape input) (at 196.85 111.76 0) (fields_autoplaced)
+    (effects (font (size 1.27 1.27)) (justify left))
   )
-  (label "EN" (at 100.33 48.26 0) (fields_autoplaced)
-    (effects (font (size 1.27 1.27)) (justify left bottom))
+  (hierarchical_label "RE&DE_RS485" (shape input) (at 208.28 123.19 180) (fields_autoplaced)
+    (effects (font (size 1.27 1.27)) (justify right))
+  )
+  (hierarchical_label "EN" (shape input) (at 82.55 92.71 180) (fields_autoplaced)
+    (effects (font (size 1.27 1.27)) (justify right))
+  )
+  (hierarchical_label "IO0" (shape input) (at 189.23 100.33 0) (fields_autoplaced)
+    (effects (font (size 1.27 1.27)) (justify left))
+  )
+  (hierarchical_label "TX0" (shape input) (at 189.23 92.71 0) (fields_autoplaced)
+    (effects (font (size 1.27 1.27)) (justify left))
+  )
+  (hierarchical_label "RXD_RS485" (shape input) (at 208.28 119.38 180) (fields_autoplaced)
+    (effects (font (size 1.27 1.27)) (justify right))
+  )
+  (hierarchical_label "LOCK_CONTROL" (shape input) (at 196.85 107.95 0) (fields_autoplaced)
+    (effects (font (size 1.27 1.27)) (justify left))
   )
   (symbol (lib_id "power:GND") (at 147.32 142.24 0) (unit 1)
