File: Microcontroller_board/Microcontroller_board.kicad_sch (KiCad schematic)
At the start: 25 parts, among them J1 USB_B_Micro, J2 Conn_01x07_Pin, Q1 BC817, Q2 BC817, SW1 SW_Reset, U1 ESP32-WROOM-E, U2 CP2102N-Axx-xQFN28

Commit message: Added peripherals to the ESP32
Connections:
- net LCD_RX2: now reaches U1.27 (GPIO16)
- net LCD_TX2: now reaches U1.28 (GPIO17)
- net ETHERNET_SS: now reaches U1.33 (GPIO21)
- net RFID_MISO renamed ETHERNET_MISO
- net RFID_MOSI renamed ETHERNET_MOSI
- net RFID_SDK renamed ETHERNET_SCK
Other:
- moved on the sheet: C3, R1
Changed lines of the file:
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@@
   (junction (at 346.71 33.02) (diameter 0) (color 0 0 0 0)
   )
-  (junction (at 260.35 68.58) (diameter 0) (color 0 0 0 0)
+  (junction (at 255.27 68.58) (diameter 0) (color 0 0 0 0)
   )
   (junction (at 40.64 74.93) (diameter 0) (color 0 0 0 0)
@@
   )
   (wire (pts (xy 171.45 80.01) (xy 177.8 80.01))
+    (stroke (width 0) (type default))
+  )
+  (wire (pts (xy 255.27 68.58) (xy 284.48 68.58))
     (stroke (width 0) (type default))
   )
@@
     (stroke (width 0) (type default))
   )
-  (wire (pts (xy 350.52 91.44) (xy 360.68 91.44))
+  (wire (pts (xy 350.52 91.44) (xy 374.65 91.44))
     (stroke (width 0) (type default))
   )
@@
     (stroke (width 0) (type default))
   )
-  (wire (pts (xy 260.35 64.77) (xy 260.35 68.58))
+  (wire (pts (xy 255.27 64.77) (xy 255.27 68.58))
     (stroke (width 0) (type default))
   )
@@
     (stroke (width 0) (type default))
   )
-  (wire (pts (xy 260.35 68.58) (xy 284.48 68.58))
-    (stroke (width 0) (type default))
-  )
-  (wire (pts (xy 254 68.58) (xy 260.35 68.58))
+  (wire (pts (xy 248.92 68.58) (xy 255.27 68.58))
     (stroke (width 0) (type default))
   )
@@
     (stroke (width 0) (type default))
   )
-  (wire (pts (xy 350.52 93.98) (xy 360.68 93.98))
+  (wire (pts (xy 350.52 93.98) (xy 374.65 93.98))
     (stroke (width 0) (type default))
   )
@@
     (stroke (width 0) (type default))
   )
-  (wire (pts (xy 260.35 68.58) (xy 260.35 71.12))
-    (stroke (width 0) (type default))
-  )
-  (wire (pts (xy 260.35 54.61) (xy 260.35 59.69))
+  (wire (pts (xy 255.27 68.58) (xy 255.27 71.12))
+    (stroke (width 0) (type default))
+  )
+  (wire (pts (xy 350.52 96.52) (xy 374.65 96.52))
+    (stroke (width 0) (type default))
+  )
+  (wire (pts (xy 255.27 54.61) (xy 255.27 59.69))
     (stroke (width 0) (type default))
   )
@@
     (stroke (width 0) (type default))
   )
-  (wire (pts (xy 350.52 101.6) (xy 360.68 101.6))
+  (wire (pts (xy 350.52 101.6) (xy 374.65 101.6))
     (stroke (width 0) (type default))
   )
@@
     (stroke (width 0) (type default))
   )
+  (wire (pts (xy 350.52 86.36) (xy 360.68 86.36))
+    (stroke (width 0) (type default))
+  )
   (wire (pts (xy 35.56 67.31) (xy 35.56 82.55))
     (stroke (width 0) (type default))
@@
     (stroke (width 0) (type default))
   )
-  (wire (pts (xy 260.35 76.2) (xy 260.35 78.74))
+  (wire (pts (xy 255.27 76.2) (xy 255.27 78.74))
     (stroke (width 0) (type default))
   )
@@
     (stroke (width 0) (type default))
   )
+  (wire (pts (xy 350.52 88.9) (xy 360.68 88.9))
+    (stroke (width 0) (type default))
+  )
   (text "ESP32" (at 224.79 26.67 0)
     (effects (font (size 7 7) (thickness 1.2) bold italic) (justify left bottom))
@@
     (effects (font (size 3 3)) (justify left bottom))
   )
+  (label "ETHERNET_MOSI" (at 374.65 101.6 0) (fields_autoplaced)
+    (effects (font (size 1.27 1.27)) (justify left bottom))
+  )
   (label "IO0" (at 204.47 86.36 0) (fields_autoplaced)
     (effects (font (size 1.27 1.27)) (justify left bottom))
@@
     (effects (font (size 1.27 1.27)) (justify left bottom))
   )
+  (label "ETHERNET_SCK" (at 374.65 91.44 0) (fields_autoplaced)
+    (effects (font (size 1.27 1.27)) (justify left bottom))
+  )
   (label "RFID_MISO" (at 360.68 93.98 0) (fields_autoplaced)
     (effects (font (size 1.27 1.27)) (justify left bottom))
@@
     (effects (font (size 1.27 1.27)) (justify left bottom))
   )
-  (label "RFID_SDK" (at 360.68 91.44 0) (fields_autoplaced)
+  (label "RFID_SCK" (at 360.68 91.44 0) (fields_autoplaced)
     (effects (font (size 1.27 1.27)) (justify left bottom))
   )
@@
     (effects (font (size 1.27 1.27)) (justify left bottom))
   )
+  (label "LCD_TX2" (at 360.68 88.9 0) (fields_autoplaced)
+    (effects (font (size 1.27 1.27)) (justify left bottom))
+  )
+  (label "ETHERNET_MISO" (at 374.65 93.98 0) (fields_autoplaced)
+    (effects (font (size 1.27 1.27)) (justify left bottom))
+  )
   (label "RTS" (at 121.92 49.53 0) (fields_autoplaced)
     (effects (font (size 1.27 1.27)) (justify left bottom))
   )
+  (label "LCD_RX2" (at 360.68 86.36 0) (fields_autoplaced)
+    (effects (font (size 1.27 1.27)) (justify left bottom))
+  )
   (label "RTS" (at 157.48 80.01 0) (fields_autoplaced)
     (effects (font (size 1.27 1.27)) (justify left bottom))
   )
+  (label "ETHERNET_SS" (at 374.65 96.52 0) (fields_autoplaced)
+    (effects (font (size 1.27 1.27)) (justify left bottom))
+  )
   (label "RX0" (at 121.92 44.45 0) (fields_autoplaced)
     (effects (font (size 1.27 1.27)) (justify left bottom))
@@
     (effects (font (size 1.27 1.27)) (justify left bottom))
   )
-  (label "EN" (at 254 68.58 0) (fields_autoplaced)
+  (label "EN" (at 248.92 68.58 0) (fields_autoplaced)
     (effects (font (size 1.27 1.27)) (justify left bottom))
   )
@@
     )
   )
-  (symbol (lib_id "Device:C_Polarized_Small") (at 260.35 73.66 0) (unit 1)
-    (in_bom yes) (on_board yes) (dnp no) (fields_autoplaced)
-    (property "Reference" "C3" (at 262.89 71.8439 0)
-      (effects (font (size 1.27 1.27)) (justify left))
-    )
-    (property "Value" "1 uF" (at 262.89 74.3839 0)
-      (effects (font (size 1.27 1.27)) (justify left))
-    )
-    (property "Footprint" "" (at 260.35 73.66 0)
-      (effects (font (size 1.27 1.27)) hide)
-    )
-    (property "Datasheet" "~" (at 260.35 73.66 0)
+  (symbol (lib_id "Device:C_Polarized_Small") (at 255.27 73.66 0) (unit 1)
+    (in_bom yes) (on_board yes) (dnp no) (fields_autoplaced)
+    (property "Reference" "C3" (at 257.81 71.8439 0)
+      (effects (font (size 1.27 1.27)) (justify left))
+    )
+    (property "Value" "1 uF" (at 257.81 74.3839 0)
+      (effects (font (size 1.27 1.27)) (justify left))
+    )
+    (property "Footprint" "" (at 255.27 73.66 0)
+      (effects (font (size 1.27 1.27)) hide)
+    )
+    (property "Datasheet" "~" (at 255.27 73.66 0)
       (effects (font (size 1.27 1.27)) hide)
     )
@@
     )
   )
-  (symbol (lib_id "power:+3.3V") (at 260.35 54.61 0) (unit 1)
-    (in_bom yes) (on_board yes) (dnp no) (fields_autoplaced)
-    (property "Reference" "#PWR04" (at 260.35 58.42 0)
-      (effects (font (size 1.27 1.27)) hide)
-    )
-    (property "Value" "+3.3V" (at 260.35 49.53 0)
-      (effects (font (size 1.27 1.27)))
-    )
-    (property "Footprint" "" (at 260.35 54.61 0)
-      (effects (font (size 1.27 1.27)) hide)
-    )
-    (property "Datasheet" "" (at 260.35 54.61 0)
+  (symbol (lib_id "power:+3.3V") (at 255.27 54.61 0) (unit 1)
+    (in_bom yes) (on_board yes) (dnp no) (fields_autoplaced)
+    (property "Reference" "#PWR04" (at 255.27 58.42 0)
+      (effects (font (size 1.27 1.27)) hide)
+    )
+    (property "Value" "+3.3V" (at 255.27 49.53 0)
+      (effects (font (size 1.27 1.27)))
+    )
+    (property "Footprint" "" (at 255.27 54.61 0)
+      (effects (font (size 1.27 1.27)) hide)
+    )
+    (property "Datasheet" "" (at 255.27 54.61 0)
       (effects (font (size 1.27 1.27)) hide)
     )
@@
     )
   )
-  (symbol (lib_id "Device:R_Small") (at 260.35 62.23 0) (unit 1)
-    (in_bom yes) (on_board yes) (dnp no) (fields_autoplaced)
-    (property "Reference" "R1" (at 262.89 60.96 0)
-      (effects (font (size 1.27 1.27)) (justify left))
-    )
-    (property "Value" "10 k" (at 262.89 63.5 0)
-      (effects (font (size 1.27 1.27)) (justify left))
-    )
-    (property "Footprint" "" (at 260.35 62.23 0)
-      (effects (font (size 1.27 1.27)) hide)
-    )
-    (property "Datasheet" "~" (at 260.35 62.23 0)
+  (symbol (lib_id "Device:R_Small") (at 255.27 62.23 0) (unit 1)
+    (in_bom yes) (on_board yes) (dnp no) (fields_autoplaced)
+    (property "Reference" "R1" (at 257.81 60.96 0)
+      (effects (font (size 1.27 1.27)) (justify left))
+    )
+    (property "Value" "10 k" (at 257.81 63.5 0)
+      (effects (font (size 1.27 1.27)) (justify left))
+    )
+    (property "Footprint" "" (at 255.27 62.23 0)
+      (effects (font (size 1.27 1.27)) hide)
+    )
+    (property "Datasheet" "~" (at 255.27 62.23 0)
       (effects (font (size 1.27 1.27)) hide)
     )
@@
     )
   )
-  (symbol (lib_id "power:GND") (at 260.35 78.74 0) (unit 1)
-    (in_bom yes) (on_board yes) (dnp no) (fields_autoplaced)
-    (property "Reference" "#PWR05" (at 260.35 85.09 0)
-      (effects (font (size 1.27 1.27)) hide)
-    )
-    (property "Value" "GND" (at 260.35 83.82 0)
-      (effects (font (size 1.27 1.27)))
-    )
-    (property "Footprint" "" (at 260.35 78.74 0)
-      (effects (font (size 1.27 1.27)) hide)
-    )
-    (property "Datasheet" "" (at 260.35 78.74 0)
-      (effects (font (size 1.27 1.27)) hide)
-    )
+  (symbol (lib_id "power:GND") (at 255.27 78.74 0) (unit 1)
+    (in_bom yes) (on_board yes) (dnp no) (fields_autoplaced)
+    (property "Reference" "#PWR05" (at 255.27 85.09 0)
+      (effects (font (size 1.27 1.27)) hide)
+    )
+    (property "Value" "GND" (at 255.27 83.82 0)
+      (effects (font (size 1.27 1.27)))
+    )
+    (property "Footprint" "" (at 255.27 78.74 0)
+      (effects (font (size 1.27 1.27)) hide)
+    )
+    (property "Datasheet" "" (at 255.27 78.74 0)
+      (effects (font (size 1.27 1.27)) hide)
+    )
