File: Microcontroller_board/Ledinterface.kicad_sch (KiCad schematic)
At the start: 0 parts

Commit message: Added led interface
Parts:
- added J1: Led_Connector, symbol Connector:Conn_01x03_Pin
- added R27: 470, symbol Device:R_Small
Connections:
- new net: J1.3 (Pin_3), R27.2
- new net +5V: J1.2 (Pin_2)
- new net GND: J1.1 (Pin_1)
- new net LED_CONTROL: R27.1
Other:
- note added: "LED RGB - WS2812b"
Changed lines of the file:
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@@
 (kicad_sch (version 20230121) (generator eeschema)
   (paper "A4")
+  (wire (pts (xy 132.08 73.66) (xy 146.05 73.66))
+    (stroke (width 0) (type default))
+  )
+  (wire (pts (xy 156.21 82.55) (xy 156.21 78.74))
+    (stroke (width 0) (type default))
+  )
+  (wire (pts (xy 156.21 78.74) (xy 162.56 78.74))
+    (stroke (width 0) (type default))
+  )
+  (wire (pts (xy 147.32 76.2) (xy 147.32 82.55))
+    (stroke (width 0) (type default))
+  )
+  (wire (pts (xy 162.56 76.2) (xy 147.32 76.2))
+    (stroke (width 0) (type default))
+  )
+  (wire (pts (xy 151.13 73.66) (xy 162.56 73.66))
+    (stroke (width 0) (type default))
+  )
+  (text "LED RGB - WS2812b" (at 20.32 30.48 0)
+    (effects (font (size 6 6) (thickness 1.2) bold italic) (justify left bottom))
+  )
+  (hierarchical_label "LED_CONTROL" (shape input) (at 132.08 73.66 180) (fields_autoplaced)
+    (effects (font (size 1.27 1.27)) (justify right))
+  )
+  (symbol (lib_id "power:+5V") (at 147.32 82.55 180) (unit 1)
+    (in_bom yes) (on_board yes) (dnp no) (fields_autoplaced)
+    (property "Reference" "#PWR022" (at 147.32 78.74 0)
+      (effects (font (size 1.27 1.27)) hide)
+    )
+    (property "Value" "+5V" (at 147.32 87.63 0)
+      (effects (font (size 1.27 1.27)))
+    )
+    (property "Footprint" "" (at 147.32 82.55 0)
+      (effects (font (size 1.27 1.27)) hide)
+    )
+    (property "Datasheet" "" (at 147.32 82.55 0)
+      (effects (font (size 1.27 1.27)) hide)
+    )
+    (pin "1")
+    (instances
+      (project "Microcontroller_board"
+        (path "/8159cf7c-7477-4d57-9227-35cab5afcf8d/7ea714e9-2b2f-44a8-989f-9a228b2aa14a"
+          (reference "#PWR022") (unit 1)
+        )
+      )
+    )
+  )
+  (symbol (lib_id "Device:R_Small") (at 148.59 73.66 90) (unit 1)
+    (in_bom yes) (on_board yes) (dnp no) (fields_autoplaced)
+    (property "Reference" "R27" (at 148.59 68.58 90)
+      (effects (font (size 1.27 1.27)))
+    )
+    (property "Value" "470" (at 148.59 71.12 90)
+      (effects (font (size 1.27 1.27)))
+    )
+    (property "Footprint" "" (at 148.59 73.66 0)
+      (effects (font (size 1.27 1.27)) hide)
+    )
+    (property "Datasheet" "~" (at 148.59 73.66 0)
+      (effects (font (size 1.27 1.27)) hide)
+    )
+    (pin "1")
+    (pin "2")
+    (instances
+      (project "Microcontroller_board"
+        (path "/8159cf7c-7477-4d57-9227-35cab5afcf8d/7ea714e9-2b2f-44a8-989f-9a228b2aa14a"
+          (reference "R27") (unit 1)
+        )
+      )
+    )
+  )
+  (symbol (lib_id "Connector:Conn_01x03_Pin") (at 167.64 76.2 180) (unit 1)
+    (in_bom yes) (on_board yes) (dnp no) (fields_autoplaced)
+    (property "Reference" "J1" (at 168.91 74.93 0)
+      (effects (font (size 1.27 1.27)) (justify right))
+    )
+    (property "Value" "Led_Connector" (at 168.91 77.47 0)
+      (effects (font (size 1.27 1.27)) (justify right))
+    )
+    (property "Footprint" "" (at 167.64 76.2 0)
+      (effects (font (size 1.27 1.27)) hide)
+    )
+    (property "Datasheet" "~" (at 167.64 76.2 0)
+      (effects (font (size 1.27 1.27)) hide)
+    )
+    (pin "1")
+    (pin "2")
+    (pin "3")
+    (instances
+      (project "Microcontroller_board"
+        (path "/8159cf7c-7477-4d57-9227-35cab5afcf8d/7ea714e9-2b2f-44a8-989f-9a228b2aa14a"
+          (reference "J1") (unit 1)
+        )
+      )
+    )
+  )
+  (symbol (lib_id "power:GND") (at 156.21 82.55 0) (unit 1)
+    (in_bom yes) (on_board yes) (dnp no) (fields_autoplaced)
+    (property "Reference" "#PWR020" (at 156.21 88.9 0)
+      (effects (font (size 1.27 1.27)) hide)
+    )
+    (property "Value" "GND" (at 156.21 87.63 0)
+      (effects (font (size 1.27 1.27)))
+    )
+    (property "Footprint" "" (at 156.21 82.55 0)
+      (effects (font (size 1.27 1.27)) hide)
+    )
+    (property "Datasheet" "" (at 156.21 82.55 0)
+      (effects (font (size 1.27 1.27)) hide)
+    )
+    (pin "1")
+    (instances
+      (project "Microcontroller_board"
+        (path "/8159cf7c-7477-4d57-9227-35cab5afcf8d/7ea714e9-2b2f-44a8-989f-9a228b2aa14a"
+          (reference "#PWR020") (unit 1)
+        )
+      )
+    )
+  )
 )
